Commit message: feat: unify the tf tree and function launch files in sim and real

File: tianracer_gazebo/urdf/tianracer.xacro (robot description, xacro)
@@ -221,5 +221,5 @@
   </joint>
   <xacro:wheel_transmission name="right_rear_wheel"/>
-  <link name="${tf_prefix}camera">
+  <link name="${tf_prefix}camera_link">
     <visual>
       <geometry>
@@ -246,5 +246,5 @@
   <joint name="camera_joint" type="fixed">
     <parent link="${tf_prefix}base_link" />
-    <child link="${tf_prefix}camera" />
+    <child link="${tf_prefix}camera_link" />
     <origin xyz="0.14851 0.0022137 0.0975" />
     <axis xyz="0 0 1" />
@@ -314,5 +314,5 @@
     <axis xyz="0 0 1" />
   </joint>
-  <link name="${tf_prefix}imu">
+  <link name="${tf_prefix}imu_link">
     <visual>
       <geometry>
@@ -338,5 +338,5 @@
   <joint name="imu_joint" type="fixed">
     <parent link="${tf_prefix}base_link" />
-    <child link="${tf_prefix}imu" />
+    <child link="${tf_prefix}imu_link" />
     <origin xyz="0 0 0.02" />
     <axis xyz="0 0 1" />
